Commit message: Add inflated bubble WSG gripper setup and floating gripper bubble environment

File: urdf/wsg50_flipped_inflated.urdf (robot description, URDF)
Before this commit: robot float_wsg50, 13 links, 12 joints
Joints:
- joint wsg50_finger_left_joint: limit lower=-0.055 upper=-0.03 effort=1.0 velocity=1.0 -> lower=-0.055 upper=0.0 effort=1.0 velocity=1.0
- joint wsg50_finger_right_joint: limit lower=0.03 upper=0.055 effort=1.0 velocity=1.0 -> lower=0.0 upper=0.055 effort=1.0 velocity=1.0
