Commit message: Add small double handle mug

File: urdf/mug_dbl.urdf (robot description, URDF)
Before this commit: robot mug_dbl.urdf, 1 links, 0 joints
Links:
- link baseLink: geometry collision mesh filename=package://meshes/mug_dbl_small.obj scale=1 1 1; visual mesh filename=package://meshes/mug_dbl_small.obj scale=1 1 1

Commit message: Add cone and filled mug models

File: urdf/mug_dbl.urdf (robot description, URDF)
Before this commit: robot mug_dbl.urdf, 1 links, 0 joints
Links:
- link baseLink: geometry collision mesh filename=package://meshes/mug_dbl_small_filled.obj scale=1 1 1; visual mesh filename=package://meshes/mug_dbl_small.obj scale=1 1 1

Commit message: Split up mug into convex decomposition as different joints

File: urdf/mug_dbl.urdf (robot description, URDF)
Before this commit: robot mug_dbl.urdf, 1 links, 0 joints
Links:
- added link link1, mass .0; collision mesh filename=package://meshes/mug_comp/mug_dbl_filled1.obj scale=1 1 1; visual mesh filename=package://meshes/mug_comp/mug_dbl_filled1.obj scale=1 1 1
- added link link10, mass .0; collision mesh filename=package://meshes/mug_comp/mug_dbl_filled10.obj scale=1 1 1; visual mesh filename=package://meshes/mug_comp/mug_dbl_filled10.obj scale=1 1 1
- added link link11, mass .0; collision mesh filename=package://meshes/mug_comp/mug_dbl_filled11.obj scale=1 1 1; visual mesh filename=package://meshes/mug_comp/mug_dbl_filled11.obj scale=1 1 1
- added link link12, mass .0; collision mesh filename=package://meshes/mug_comp/mug_dbl_filled12.obj scale=1 1 1; visual mesh filename=package://meshes/mug_comp/mug_dbl_filled12.obj scale=1 1 1
- added link link13, mass .0; collision mesh filename=package://meshes/mug_comp/mug_dbl_filled13.obj scale=1 1 1; visual mesh filename=package://meshes/mug_comp/mug_dbl_filled13.obj scale=1 1 1
- added link link14, mass .0; collision mesh filename=package://meshes/mug_comp/mug_dbl_filled14.obj scale=1 1 1; visual mesh filename=package://meshes/mug_comp/mug_dbl_filled14.obj scale=1 1 1
- added link link2, mass .0; collision mesh filename=package://meshes/mug_comp/mug_dbl_filled2.obj scale=1 1 1; visual mesh filename=package://meshes/mug_comp/mug_dbl_filled2.obj scale=1 1 1
- added link link3, mass .0; collision mesh filename=package://meshes/mug_comp/mug_dbl_filled3.obj scale=1 1 1; visual mesh filename=package://meshes/mug_comp/mug_dbl_filled3.obj scale=1 1 1
- added link link4, mass .0; collision mesh filename=package://meshes/mug_comp/mug_dbl_filled4.obj scale=1 1 1; visual mesh filename=package://meshes/mug_comp/mug_dbl_filled4.obj scale=1 1 1
- added link link5, mass .0; collision mesh filename=package://meshes/mug_comp/mug_dbl_filled5.obj scale=1 1 1; visual mesh filename=package://meshes/mug_comp/mug_dbl_filled5.obj scale=1 1 1
- added link link6, mass .0; collision mesh filename=package://meshes/mug_comp/mug_dbl_filled6.obj scale=1 1 1; visual mesh filename=package://meshes/mug_comp/mug_dbl_filled6.obj scale=1 1 1
- added link link7, mass .0; collision mesh filename=package://meshes/mug_comp/mug_dbl_filled7.obj scale=1 1 1; visual mesh filename=package://meshes/mug_comp/mug_dbl_filled7.obj scale=1 1 1
- added link link8, mass .0; collision mesh filename=package://meshes/mug_comp/mug_dbl_filled8.obj scale=1 1 1; visual mesh filename=package://meshes/mug_comp/mug_dbl_filled8.obj scale=1 1 1
- added link link9, mass .0; collision mesh filename=package://meshes/mug_comp/mug_dbl_filled9.obj scale=1 1 1; visual mesh filename=package://meshes/mug_comp/mug_dbl_filled9.obj scale=1 1 1
- link baseLink: geometry collision mesh filename=package://meshes/mug_comp/mug_dbl_filled.obj scale=1 1 1; visual mesh filename=package://meshes/mug_comp/mug_dbl.obj scale=1 1 1
Joints:
- added joint joint1: type fixed, parent baseLink, child link1, origin xyz=0 0 0 rpy=0 0 0
- added joint joint10: type fixed, parent baseLink, child link10, origin xyz=0 0 0 rpy=0 0 0
- added joint joint11: type fixed, parent baseLink, child link11, origin xyz=0 0 0 rpy=0 0 0
- added joint joint12: type fixed, parent baseLink, child link12, origin xyz=0 0 0 rpy=0 0 0
- added joint joint13: type fixed, parent baseLink, child link13, origin xyz=0 0 0 rpy=0 0 0
- added joint joint14: type fixed, parent baseLink, child link14, origin xyz=0 0 0 rpy=0 0 0
- added joint joint2: type fixed, parent baseLink, child link2, origin xyz=0 0 0 rpy=0 0 0
- added joint joint3: type fixed, parent baseLink, child link3, origin xyz=0 0 0 rpy=0 0 0
- added joint joint4: type fixed, parent baseLink, child link4, origin xyz=0 0 0 rpy=0 0 0
- added joint joint5: type fixed, parent baseLink, child link5, origin xyz=0 0 0 rpy=0 0 0
- added joint joint6: type fixed, parent baseLink, child link6, origin xyz=0 0 0 rpy=0 0 0
- added joint joint7: type fixed, parent baseLink, child link7, origin xyz=0 0 0 rpy=0 0 0
- added joint joint8: type fixed, parent baseLink, child link8, origin xyz=0 0 0 rpy=0 0 0
- added joint joint9: type fixed, parent baseLink, child link9, origin xyz=0 0 0 rpy=0 0 0
