Commit message: Add small mug object

File: urdf/mug_dbl_small.urdf (robot description, URDF)
Before this commit: robot mug_dbl.urdf, 1 links, 0 joints
Links:
- added link link1, mass .0; collision mesh filename=package://meshes/mug_small_comp/handle1.obj scale=1 1 1; visual mesh filename=package://meshes/mug_small_comp/handle1.obj scale=1 1 1
- added link link10, mass .0; collision mesh filename=package://meshes/mug_small_comp/handle10.obj scale=1 1 1; visual mesh filename=package://meshes/mug_small_comp/handle10.obj scale=1 1 1
- added link link11, mass .0; collision mesh filename=package://meshes/mug_small_comp/handle11.obj scale=1 1 1; visual mesh filename=package://meshes/mug_small_comp/handle11.obj scale=1 1 1
- added link link12, mass .0; collision mesh filename=package://meshes/mug_small_comp/handle12.obj scale=1 1 1; visual mesh filename=package://meshes/mug_small_comp/handle12.obj scale=1 1 1
- added link link13, mass .0; collision mesh filename=package://meshes/mug_small_comp/handle13.obj scale=1 1 1; visual mesh filename=package://meshes/mug_small_comp/handle13.obj scale=1 1 1
- added link link14, mass .0; collision mesh filename=package://meshes/mug_small_comp/handle14.obj scale=1 1 1; visual mesh filename=package://meshes/mug_small_comp/handle14.obj scale=1 1 1
- added link link2, mass .0; collision mesh filename=package://meshes/mug_small_comp/handle2.obj scale=1 1 1; visual mesh filename=package://meshes/mug_small_comp/handle2.obj scale=1 1 1
- added link link3, mass .0; collision mesh filename=package://meshes/mug_small_comp/handle3.obj scale=1 1 1; visual mesh filename=package://meshes/mug_small_comp/handle3.obj scale=1 1 1
- added link link4, mass .0; collision mesh filename=package://meshes/mug_small_comp/handle4.obj scale=1 1 1; visual mesh filename=package://meshes/mug_small_comp/handle4.obj scale=1 1 1
- added link link5, mass .0; collision mesh filename=package://meshes/mug_small_comp/handle5.obj scale=1 1 1; visual mesh filename=package://meshes/mug_small_comp/handle5.obj scale=1 1 1
- added link link6, mass .0; collision mesh filename=package://meshes/mug_small_comp/handle6.obj scale=1 1 1; visual mesh filename=package://meshes/mug_small_comp/handle6.obj scale=1 1 1
- added link link7, mass .0; collision mesh filename=package://meshes/mug_small_comp/handle7.obj scale=1 1 1; visual mesh filename=package://meshes/mug_small_comp/handle7.obj scale=1 1 1
- added link link8, mass .0; collision mesh filename=package://meshes/mug_small_comp/handle8.obj scale=1 1 1; visual mesh filename=package://meshes/mug_small_comp/handle8.obj scale=1 1 1
- added link link9, mass .0; collision mesh filename=package://meshes/mug_small_comp/handle9.obj scale=1 1 1; visual mesh filename=package://meshes/mug_small_comp/handle9.obj scale=1 1 1
- link baseLink: geometry collision mesh filename=package://meshes/mug_small_comp/filled_base.obj scale=1 1 1; visual mesh filename=package://meshes/mug_small_comp/unfilled_base.obj scale=1 1 1
Joints:
- added joint joint1: type fixed, parent baseLink, child link1, origin xyz=0 0 0 rpy=0 0 0
- added joint joint10: type fixed, parent baseLink, child link10, origin xyz=0 0 0 rpy=0 0 0
- added joint joint11: type fixed, parent baseLink, child link11, origin xyz=0 0 0 rpy=0 0 0
- added joint joint12: type fixed, parent baseLink, child link12, origin xyz=0 0 0 rpy=0 0 0
- added joint joint13: type fixed, parent baseLink, child link13, origin xyz=0 0 0 rpy=0 0 0
- added joint joint14: type fixed, parent baseLink, child link14, origin xyz=0 0 0 rpy=0 0 0
- added joint joint2: type fixed, parent baseLink, child link2, origin xyz=0 0 0 rpy=0 0 0
- added joint joint3: type fixed, parent baseLink, child link3, origin xyz=0 0 0 rpy=0 0 0
- added joint joint4: type fixed, parent baseLink, child link4, origin xyz=0 0 0 rpy=0 0 0
- added joint joint5: type fixed, parent baseLink, child link5, origin xyz=0 0 0 rpy=0 0 0
- added joint joint6: type fixed, parent baseLink, child link6, origin xyz=0 0 0 rpy=0 0 0
- added joint joint7: type fixed, parent baseLink, child link7, origin xyz=0 0 0 rpy=0 0 0
- added joint joint8: type fixed, parent baseLink, child link8, origin xyz=0 0 0 rpy=0 0 0
- added joint joint9: type fixed, parent baseLink, child link9, origin xyz=0 0 0 rpy=0 0 0
