Commit message: Add cracker box and virtual mass to avoid toppling instead of lateral friction

File: urdf/YcbPowerDrillZeroed/model.urdf (robot description, URDF)
Before this commit: robot model.urdf, 1 links, 0 joints
Links:
- added link virtualMassLink, mass 8.0; visual box size=0.01 0.01 0.01
Joints:
- added joint virtualMassJoint: type fixed, parent baseLink, child virtualMassLink, origin xyz=0.0 0.0 -0.4 rpy=0 0 0
